File: protoboard.sch (KiCad schematic (older format))
At the start: 60 parts, among them U1 PROTO_SOIC6, U10 PROTO_SOT23, U11 PROTO_SOIC6, U12 PROTO_SOT23, U13 PROTO_SOIC6, U14 PROTO_SOT23, U15 PROTO_SOIC6, U16 PROTO_SOT23, U17 PROTO_SOIC6, U18 PROTO_SOT23, U19 PROTO_SOIC6, U2 PROTO_SOT23, U20 PROTO_SOT23, U21 PROTO_SOIC6, U22 PROTO_SOT23, U23 PROTO_SOIC6, U24 PROTO_SOT23, U3 PROTO_SOIC6, U30 PAD, U31 PAD, U32 PAD, U33 PAD, U34 PAD, U35 PAD, U36 PAD, U37 PAD, U38 PAD, U39 PAD, U4 PROTO_SOT23, U40 PAD, U41 PAD, U42 PAD, U43 PAD, U44 PAD, U45 PAD, U46 PAD, U47 PAD, U48 PAD, U49 PAD, U5 PROTO_SOIC6, U50 PAD, U51 PAD, U52 PAD, U53 PAD, U54 PAD, U55 PAD, U56 PAD, U57 PAD, U58 PAD, U59 PAD, U6 PROTO_SOT23, U60 PAD, U61 PAD, U62 PAD, U63 PAD, U64 PAD, U65 PAD, U7 PROTO_SOIC6, U8 PROTO_SOT23, U9 PROTO_SOIC6

Commit message: Add more pads
Parts:
- added P1, P10, P11, P12, P13, P14, P15, P16, P17, P18, P19, P2, P20, P21, P22, P23, P24, P25, P26, P27, P28, P29, P3, P30, P31, P32, P33, P34, P35, P36, P4, P5, P6, P7, P8, P9: PAD, proto_pad2, symbol PAD
- added U100, U1001, U101, U102, U103, U104, U105, U106, U107, U108, U109, U110, U111, U112, U113, U114, U115, U116, U117, U118, U119, U120, U121, U122, U123, U124, U125, U126, U127, U128, U129, U130, U131, U132, U133, U134, U135, U136, U137, U138, U139, U140, U141, U142, U143, U144, U145, U146, U147, U148, U149, U150, U151, U152, U153, U154, U155, U156, U157, U158, U159, U160, U161, U162, U163, U164, U165, U166, U167, U168, U25, U26, U27, U28, U29, U66, U67, U68, U69, U70, U71, U72, U73, U74, U75, U76, U77, U78, U79, U80, U81, U82, U83, U84, U85, U86, U87, U88, U89, U90, U91, U92, U93, U94, U95, U96, U97, U98, U99: PAD, proto_pad, symbol PAD
Connections:
- new net: U100.1, U101.1, U66.1, U67.1, U68.1, U69.1, U70.1, U71.1, U72.1, U73.1, U74.1, U75.1, U76.1, U77.1, U78.1, U79.1, U80.1, U81.1, U82.1, U83.1, U84.1, U85.1, U86.1, U87.1, U88.1, U89.1, U90.1, U91.1, U92.1, U93.1, U94.1, U95.1, U96.1, U97.1, U98.1, U99.1
- new net: U102.1, U103.1, U104.1, U105.1, U106.1, U107.1, U108.1, U109.1, U110.1, U111.1, U112.1, U113.1, U114.1, U115.1, U116.1, U117.1, U118.1, U119.1, U120.1, U121.1, U122.1, U123.1, U124.1, U125.1, U126.1, U127.1, U128.1, U129.1, U130.1, U131.1, U132.1, U25.1, U26.1, U27.1, U28.1, U29.1
- new net: U133.1, U134.1, U135.1, U136.1, U137.1, U138.1, U139.1, U140.1, U141.1, U142.1, U143.1, U144.1, U145.1, U146.1, U147.1, U148.1, U149.1, U150.1, U151.1, U152.1, U153.1, U154.1, U155.1, U156.1, U157.1, U158.1, U159.1, U160.1, U161.1, U162.1, U163.1, U164.1, U165.1, U166.1, U167.1, U168.1

Commit message: Populate board with a lot of pads
Parts:
- removed P1, P16, P17, P2, P36, P8: PAD, proto_pad2, symbol PAD
- added H1, H2, H3, H4: HOLE, hole_2mm, symbol HOLE
- added PT1, PT10, PT11, PT12, PT13, PT14, PT15, PT16, PT17, PT18, PT19, PT2, PT20, PT21, PT22, PT23, PT24, PT25, PT26, PT27, PT28, PT29, PT3, PT30, PT31, PT32, PT33, PT34, PT35, PT36, PT37, PT38, PT39, PT4, PT40, PT41, PT42, PT43, PT44, PT45, PT46, PT47, PT48, PT49, PT5, PT50, PT51, PT52, PT53, PT54, PT55, PT56, PT57, PT58, PT59, PT6, PT60, PT61, PT62, PT63, PT64, PT7, PT8, PT9, U1000, U1002, U1003, U1004, U1005, U1006, U1007, U169, U170, U171, U172, U173, U174, U175, U176, U177, U178, U179, U180, U181, U182, U183, U184, U185, U186, U187, U188, U189, U190, U191, U192, U193, U194, U195, U196, U197, U198, U199, U200, U201, U202, U203, U204, U205, U206, U207, U208, U209, U210, U211, U212, U213, U214, U215, U216, U217, U218, U219, U220, U221, U222, U223, U224, U225, U226, U227, U228, U229, U230, U231, U232, U233, U234, U235, U236, U237, U238, U239, U240, U241, U242, U243, U244, U245, U246, U247, U248, U249, U250, U251, U252, U253, U254, U255, U256, U257, U258, U259, U260, U261, U262, U263, U264, U265, U266, U267, U268, U269, U270, U271, U272, U273, U274, U275, U276, U277, U278, U279, U280, U281, U282, U283, U284, U285, U286, U287, U288, U289, U290, U291, U292, U293, U294, U295, U296, U297, U298, U299, U300, U301, U302, U303, U304, U305, U306, U307, U308, U309, U310, U311, U312, U313, U314, U315, U316, U317, U318, U319, U320, U321, U322, U323, U324, U325, U326, U327, U328, U329, U330, U331, U332, U333, U334, U335, U336, U337, U338, U339, U340, U341, U342, U343, U344, U345, U346, U347, U348, U349, U350, U351, U352, U353, U354, U355, U356, U357, U358, U359, U360, U361, U362, U363, U364, U365, U366, U367, U368, U369, U370, U371, U372, U373, U374, U375, U376, U377, U378, U379, U380, U381, U382, U383, U384, U385, U386, U387, U388, U389, U390, U391, U392, U393, U394, U395, U396, U397, U398, U399, U400, U401, U402, U403, U404, U405, U406, U407, U408, U409, U410, U411, U412, U413, U414, U415, U416, U417, U418, U419, U420, U421, U422, U423, U424, U425, U426, U427, U428, U429, U430, U431, U432, U433, U434, U435, U436, U437, U438, U439, U440, U441, U442, U443, U444, U445, U446, U447, U448, U449, U450, U451, U452, U453, U454, U455, U456, U457, U458, U459, U460, U461, U462, U463, U464, U465, U466, U467, U468, U469, U470, U471, U472, U473, U474, U475, U476, U477, U478, U479, U480, U481, U482, U483, U484, U485, U486, U487, U488, U489, U490, U491, U492, U493, U494, U495, U496, U497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: PAD, proto_pad, symbol PAD
- added TQFP1: PROTO_TQFP64, proto_tqfp_08, symbol PROTO_TQFP64
Connections:
- new net: PT1.1, TQFP1.1
- new net: PT10.1, TQFP1.10
- new net: PT11.1, TQFP1.11
- new net: PT12.1, TQFP1.12
- new net: PT13.1, TQFP1.13
- new net: PT14.1, TQFP1.14
- new net: PT15.1, TQFP1.15
- new net: PT16.1, TQFP1.16
- new net: PT17.1, TQFP1.17
- new net: PT18.1, TQFP1.18
- new net: PT19.1, TQFP1.19
- new net: PT2.1, TQFP1.2
- new net: PT20.1, TQFP1.20
- new net: PT21.1, TQFP1.21
- new net: PT22.1, TQFP1.22
- new net: PT23.1, TQFP1.23
- new net: PT24.1, TQFP1.24
- new net: PT25.1, TQFP1.25
- new net: PT26.1, TQFP1.26
- new net: PT27.1, TQFP1.27
- new net: PT28.1, TQFP1.28
- new net: PT29.1, TQFP1.29
- new net: PT3.1, TQFP1.3
- new net: PT30.1, TQFP1.30
- new net: PT31.1, TQFP1.31
- new net: PT32.1, TQFP1.32
- new net: PT33.1, TQFP1.33
- new net: PT34.1, TQFP1.34
- new net: PT35.1, TQFP1.35
- new net: PT36.1, TQFP1.36
- new net: PT37.1, TQFP1.37
- new net: PT38.1, TQFP1.38
- new net: PT39.1, TQFP1.39
- new net: PT4.1, TQFP1.4
- new net: PT40.1, TQFP1.40
- new net: PT41.1, TQFP1.41
- new net: PT42.1, TQFP1.42
- new net: PT43.1, TQFP1.43
- new net: PT44.1, TQFP1.44
- new net: PT45.1, TQFP1.45
- new net: PT46.1, TQFP1.46
- new net: PT47.1, TQFP1.47
- new net: PT48.1, TQFP1.48
- new net: PT49.1, TQFP1.49
- new net: PT5.1, TQFP1.5
- new net: PT50.1, TQFP1.50
- new net: PT51.1, TQFP1.51
- new net: PT52.1, TQFP1.52
- new net: PT53.1, TQFP1.53
- new net: PT54.1, TQFP1.54
- new net: PT55.1, TQFP1.55
- new net: PT56.1, TQFP1.56
- new net: PT57.1, TQFP1.57
- new net: PT58.1, TQFP1.58
- new net: PT59.1, TQFP1.59
- new net: PT6.1, TQFP1.6
- new net: PT60.1, TQFP1.60
- new net: PT61.1, TQFP1.61
- new net: PT62.1, TQFP1.62
- new net: PT63.1, TQFP1.63
- new net: PT64.1, TQFP1.64
- new net: PT7.1, TQFP1.7
- new net: PT8.1, TQFP1.8
- new net: PT9.1, TQFP1.9
Other:
- moved on the sheet: P10, P11, P12, P13, P14, P15, P18, P19, P20, P21, P22, P23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

Commit message: Add a bunch of pads Dual row of header pads
Parts:
- added P1, P16, P17, P2, P36, P37, P38, P39, P40, P41, P42, P43, P44, P45, P8: PAD, proto_pad2, symbol PAD
- added U1008, U1009, U1010, U1011, U1012, U1013, U1014, U1015, U1016, U1017, U1018, U1019, U1020, U1021, U1022, U1023, U1024, U1025, U1026, U1027, U1028, U1029, U1030, U1031, U1032, U1033, U1034, U1035, U1036, U1037, U1038, U1039, U1040, U1041, U1042, U1043, U1044, U1045, U1046, U1047, U1048, U1049, U1050, U1051, U1052, U1053, U1054, U1055, U1056, U1057, U1058, U1059, U1060, U1061, U1062, U1063, U1064, U1065, U1066, U1067, U1068, U1069, U1070, U1071, U1072, U1073, U1074, U1075, U1076, U1077, U1078, U1079, U1080, U1081, U1082, U1083, U1084, U1085, U1086, U1087, U1088, U1089, U1090, U1091, U1092, U1093, U1094, U1095, U1096, U1097, U1098, U1099, U1100, U1101, U1102, U1103, U1104, U1105, U1106, U1107, U1108, U1109, U1110, U1111, U1112, U1113, U1114, U1115, U1116, U1117, U1118, U1119, U1120, U1121, U1122, U1123, U1124, U1125, U1126, U1127, U1128, U1129, U1130, U1131, U1132, U1133, U1134, U1135, U1136, U1137, U1138, U1139, U1140, U1141, U1142, U1143, U1144, U1145, U1146, U1147, U1148, U1149, U1150, U1151, U1152, U1153, U1154, U1155, U1156, U1157, U1158, U1159, U1160, U1161, U1162, U1163, U1164, U1165, U1166, U1167, U1168, U1169, U1170, U1171, U1172, U1173, U1174, U1175, U1176, U1177, U1178, U1179, U1180, U1181, U1182, U1183, U1184, U1185, U1186, U1187, U1188, U1189, U1190, U1191, U1192, U1193, U1194, U1195, U1196, U1197, U1198, U1199, U1200, U1201, U1202, U1203, U1204, U1205, U1206, U1207, U1208, U1209, U1210, U1211, U1212, U1213, U1214, U1215, U1216, U1217, U1218, U1219, U1220, U1221, U1222, U1223, U1224, U1225, U1226, U1227, U1228, U1229, U1230, U1231, U1232, U1233, U1234, U1235, U1236, U1237, U1238, U1239, U1240, U1241, U1242, U1243, U1244, U1245, U1246, U1247, U1248, U1249, U1250, U1251, U1252, U1253, U1254, U1255, U1256, U1257, U1258, U1259, U1260, U1261, U1262, U1263, U1264, U1265, U1266, U1267, U1268, U1269, U1270, U1271, U1272, U1273, U1274, U1275, U1276, U1277, U1278, U1279, U1280, U1281, U1282, U1283, U1284, U1285, U1286, U1287, U1288, U1289, U1290, U1291, U1292, U1293, U1294, U1295, U1296, U1297, U1298, U1299, U1300, U1301, U1302, U1303, U1304, U1305, U1306, U1307, U1308, U1309, U1310, U1311, U1312, U1313, U1314, U1315, U1316, U1317, U1318, U1319, U1320, U1321, U1322, U1323, U1324, U1325, U1326, U1327, U1328, U1329, U1330, U1331, U1332: PAD, proto_pad, symbol PAD

Commit message: All pads here
Parts:
- added U1333, U1334, U1335, U1336, U1337, U1338, U1339, U1340, U1341, U1342, U1343, U1344, U1345, U1346, U1347, U1348, U1349, U1350, U1351, U1352, U1353, U1354, U1355, U1356, U1357, U1358, U1359, U1360, U1361, U1362, U1363, U1364, U1365, U1366, U1367, U1368, U1369, U1370, U1371, U1372, U1373, U1374, U1375, U1376, U1377, U1378, U1379, U1380, U1381, U1382, U1383, U1384, U1385, U1386, U1387, U1388, U1389, U1390, U1391, U1392, U1393, U1394, U1395, U1396, U1397, U1398, U1399, U1400, U1401, U1402, U1403, U1404, U1405, U1406, U1407, U1408, U1409, U1410, U1411, U1412, U1413, U1414, U1415, U1416, U1417, U1418, U1419, U1420, U1421, U1422, U1423, U1424, U1425, U1426, U1427, U1428, U1429, U1430, U1431, U1432, U1433, U1434, U1435, U1436, U1437, U1438, U1439, U1440, U1441, U1442, U1443, U1444, U1445, U1446, U1447, U1448, U1449, U1450, U1451, U1452, U1453, U1454, U1455, U1456, U1457, U1458, U1459, U1460, U1461, U1462, U1463, U1464, U1465, U1466, U1467, U1468, U1469, U1470, U1471, U1472, U1473, U1474, U1475, U1476, U1477, U1478, U1479, U1480, U1481, U1482, U1483, U1484, U1485, U1486, U1487, U1488, U1489, U1490, U1491, U1492, U1493, U1494, U1495, U1496, U1497, U1498, U1499, U1500, U1501, U1502, U1503, U1504, U1505, U1506, U1507, U1508, U1509, U1510, U1511, U1512, U1513, U1514, U1515, U1516, U1517, U1518, U1519, U1520, U1521, U1522, U1523, U1524, U1525, U1526, U1527, U1528, U1529, U1530, U1531, U1532, U1533, U1534, U1535, U1536, U1537, U1538, U1539, U1540, U1541, U1542, U1543, U1544, U1545, U1546, U1547, U1548, U1549, U1550, U1551, U1552, U1553, U1554, U1555, U1556, U1557, U1558, U1559, U1560, U1561, U1562, U1563, U1564, U1565, U1566, U1567, U1568, U1569, U1570, U1571, U1572, U1573, U1574, U1575, U1576, U1577, U1578, U1579, U1580, U1581, U1582, U1583, U1584, U1585, U1586, U1587, U1588, U1589, U1590, U1591, U1592, U1593, U1594, U1595, U1596, U1597, U1598, U1599, U1600, U1601, U1602, U1603, U1604, U1605, U1606, U1607, U1608, U1609, U1610, U1611, U1612, U1613, U1614, U1615, U1616, U1617, U1618, U1619, U1620, U1621, U1622, U1623, U1624, U1625, U1626, U1627, U1628, U1629, U1630, U1631, U1632, U1633, U1634, U1635, U1636, U1637, U1638, U1639, U1640, U1641, U1642, U1643, U1644, U1645, U1646, U1647, U1648, U1649, U1650, U1651, U1652, U1653, U1654, U1655, U1656, U1657, U1658, U1659, U1660, U1661, U1662, U1663, U1664, U1665, U1666, U1667, U1668, U1669, U1670, U1671, U1672, U1673, U1674, U1675, U1676, U1677, U1678, U1679, U1680, U1681, U1682, U1683, U1684, U1685, U1686, U1687, U1688, U1689, U1690, U1691, U1692, U1693, U1694, U1695, U1696, U1697, U1698, U1699, U1700, U1701, U1702, U1703, U1704, U1705, U1706, U1707, U1708, U1709, U1710, U1711, U1712, U1713, U1714, U1715, U1716, U1717, U1718, U1719, U1720, U1721, U1722, U1723, U1724, U1725, U1726, U1727, U1728, U1729, U1730, U1731, U1732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: PAD, proto_pad, symbol PAD

Commit message: Make board fit into 5x5cm
Parts:
- removed U1107, U1109, U1298, U1305, U1312, U1321, U1327, U1328, U1339, U1340, U1346, U1347, U1350, U1351, U1359, U1360, U1363, U1365, U1366, U1377, U1378, U1381, U1382, U1383, U1389, U1392, U1393, U1395, U1404, U1405, U1407, U1408, U1413, U1415, U1428, U1429, U1431, U1432, U1433, U1434, U1454, U1458, U1459, U1463, U1464, U1465, U1466, U1468, U1469, U1472, U1473, U1474, U1475, U1476, U1477, U1478, U1479, U1480, U1645, U1654, U1670, U1673, U1678, U1696, U1697, U1720, U1722, U1730, U1742, U1753, U1755, U1764, U1766, U1768, U1769, U1770, U1771, U180, U188, U195, U205, U214, U221, U224, U254, U260, U261, U272, U280, U293, U300, U313, U320, U330, U344, U345, U363, U464, U468, U493, U495, U510, U557, U560, U574, U575, U579, U580, U581, U582, U590, U591, U592, U593, U594, U628, U635, U648, U653, U654, U656, U669, U672, U673, U728, U732, U733, U736, U737, U738, U743, U746, U751, U756, U757, U761, U762, U772, U775, U776, U784, U789, U792, U793, U807, U810, U824, U827, U835, U838, U850, U852, U858, U863: PAD, proto_pad, symbol PAD
